Commit message: DC motors Control | Roboclaw

File: dicerox_arm_confv2/urdf/DICEROX_ARM.urdf (robot description, URDF)
Before this commit: robot dicer_arm_confv2, 7 links, 6 joints
Joints:
- joint Joint2: limit lower=-1.5708 upper=1.5708 effort=100 velocity=100 -> lower=-4.18879 upper=0.00000 effort=100 velocity=100; origin xyz=0 -0.017 0.1165 rpy=1.5708 0 0 -> xyz=0 -0.017 0.1165 rpy=1.5708 -1.5708 0
- joint Joint3: limit lower=-1.5708 upper=1.5708 effort=100 velocity=100 -> lower=0.00000 upper=3.40339 effort=100 velocity=100; origin xyz=0.056326 0.43175 0 rpy=0 0 1.5708 -> xyz=0.056326 0.43175 0 rpy=0 0 0.2
